File: TEST V1/TEST V1.kicad_sch (KiCad schematic)
At the start: 60 parts, among them IC1 W25Q16JVUXIQ, J1 Conn_01x16_Socket, J2 USB_C_Receptacle_USB2.0_14P, J3 Conn_01x03_Socket, SW1 SW_Push_SPDT, SW2 SW_Push_SPDT, U1 RP2040, U2 SN74LVC244APWT, U3 74AHCT125, Y1 Crystal_12MHz

Commit message: updated RPS schematic
Other:
- sheet RPS renamed RPS & POWER DESIGN
- removed sheet POWER SUPPLY
- sheet RPS & POWER DESIGN: file RPS.kicad_sch -> RPS&pwr.kicad_sch
