File: TEST V1/TEST V1.kicad_sch (KiCad schematic)
At the start: 60 parts, among them IC1 W25Q16JVUXIQ, J1 Conn_01x16_Socket, J2 USB_C_Receptacle_USB2.0_14P, J3 Conn_01x03_Socket, SW1 SW_Push_SPDT, SW2 SW_Push_SPDT, U1 RP2040, U2 SN74LVC244APWT, U3 74AHCT125, Y1 Crystal_12MHz

Commit message: all updated
Parts:
- removed C9: 100n, Capacitor_SMD:C_0603_1608Metric_Pad1.08x0.95mm_HandSolder, symbol Device:C
- removed R10, R11, R12, R13, R7, R8, R9: 0R, Resistor_SMD:R_0603_1608Metric_Pad0.98x0.95mm_HandSolder, symbol Device:R
- removed R19: 0, Resistor_SMD:R_0603_1608Metric_Pad0.98x0.95mm_HandSolder, symbol Device:R
- removed SW1, SW2: SW_Push_SPDT, symbol Switch:SW_Push_SPDT
- removed U1: RP2040, Package_DFN_QFN:QFN-56-1EP_7x7mm_P0.4mm_EP3.2x3.2mm, symbol MCU_RaspberryPi_New:RP2040
- removed U2: SN74LVC244APWT, SN74LVC244APWT:SOP65P640X120-20N, symbol SN74LVC244APWT:SN74LVC244APWT
- added C43: 100n, Capacitor_SMD:C_0603_1608Metric_Pad1.08x0.95mm_HandSolder, symbol Device:C
- added J14, J15: Conn_01x02_Pin, Connector_PinHeader_2.54mm:PinHeader_1x02_P2.54mm_Vertical, symbol Connector:Conn_01x02_Pin
- added R60: 0, Resistor_SMD:R_0603_1608Metric_Pad0.98x0.95mm_HandSolder, symbol Device:R
- added U13: RP2040, Package_DFN_QFN:QFN-56-1EP_7x7mm_P0.4mm_EP3.2x3.2mm, symbol MCU_RaspberryPi:RP2040
- added U14: SN74LVC244APWT, SN74LVC244APWT:SOP65P640X120-20N, symbol SN74LVC244APWT:SN74LVC244APWT
Connections:
- net GPIO0 is gone; now on net GPIO8: U3.2
- net GPIO1 is gone; now on net GPIO9: U3.5
- net GPIO2 is gone; now on net GPIO10: U3.9
- net GPIO3 is gone; now on net GPIO11: U3.12
- net +1V1: now also U13.45 (VREG_VOUT)
- net +3.3V: now also R60.1
- net ADC_AVDD: now also U13.43 (ADC_AVDD)
- net DVDD: now also U13.23 (DVDD), U13.50 (DVDD)
- net GND: now also C1.1, C43.2, J14.2 (Pin_2), J15.2 (Pin_2), U13.19 (TESTEN), U13.57 (GND), U14.1 (~{1OE}), U14.10 (GND), U14.19 (~{2OE}); no longer C1.2
- net GPIO10: now also U13.13 (GPIO10)
- net GPIO11: now also U13.14 (GPIO11)
- net GPIO24: now also U13.36 (GPIO24)
- net GPIO8: now also U13.11 (GPIO8)
- net GPIO9: now also U13.12 (GPIO9)
- net I2C_SCL: now also U13.16 (GPIO13)
- net I2C_SDA: now also U13.15 (GPIO12)
- net LA0_IN: now also U14.2 (1A1)
- net LA1_IN: now also U14.4 (1A2)
- net LA2_IN: now also U14.6 (1A3)
- net LA3_IN: now also U14.8 (1A4)
- net LA4_IN: now also U14.11 (2A1)
- net LA5_IN: now also U14.13 (2A2)
- net LA6_IN: now also U14.15 (2A3)
- net LA7_IN: now also U14.17 (2A4)
- net QSPI_CSN: now also U13.56 (QSPI_SS)
- net QSPI_SCLK: now also U13.52 (QSPI_SCLK)
- net QSPI_SD0: now also U13.53 (QSPI_SD0)
- net QSPI_SD1: now also U13.55 (QSPI_SD1)
- net QSPI_SD2: now also U13.54 (QSPI_SD2)
- net QSPI_SD3: now also U13.51 (QSPI_SD3)
- net RUN: now also J14.1 (Pin_1), U13.26 (RUN)
- net SPI_EN: now also U13.28 (GPIO17)
- net SPI_MOSI: now also U13.30 (GPIO19)
- net SPI_SCLK: now also U13.29 (GPIO18)
- net SWCLK: now also U13.24 (SWCLK)
- net SWD: now also U13.25 (SWD)
- net USB_DM: now also R6.2; no longer R5.2
- net USB_DP: now also R5.2; no longer R6.2
- net XIN: now also U13.20 (XIN)
- net XOUT: now also U13.21 (XOUT)
- net at R2.2: now also J15.1 (Pin_1)
- net at R6.1: now also U13.46 (USB_DM)
- net at R5.1: now also U13.47 (USB_DP)
- net at C6.1, R15.1: now also U13.44 (VREG_IN)
- net at C2.1, IC1.8 (VCC), R1.2: now also C1.2; no longer C1.1
- net IOVDD: no longer names the net of C10.1, C11.1, C12.1, C13.1, C7.1, C8.1, R18.2
- net IOVDD: now also U13.1 (IOVDD), U13.10 (IOVDD), U13.22 (IOVDD), U13.33 (IOVDD), U13.42 (IOVDD), U13.48 (USB_VDD), U13.49 (IOVDD)
- new net: U13.5 (GPIO3), U14.12 (1Y4)
- new net: U13.4 (GPIO2), U14.14 (1Y3)
- new net: U13.3 (GPIO1), U14.16 (1Y2)
- new net: U13.2 (GPIO0), U14.18 (1Y1)
- new net: C43.1, R60.2, U14.20 (VCC)
- new net: U13.9 (GPIO7), U14.3 (2Y4)
- new net: U13.8 (GPIO6), U14.5 (2Y3)
- new net: U13.7 (GPIO5), U14.7 (2Y2)
- new net: U13.6 (GPIO4), U14.9 (2Y1)
- no-connect marks 5 -> 14
Other:
- note removed: "DECOUPLING CAPS"
- moved on the sheet: C1, C10, C11, C12, C13, C14, C15, C2, C3, C4, C5, C6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
