File: TEST V1/TEST V1.kicad_sch (KiCad schematic)
At the start: 53 parts, among them IC1 W25Q16JVUXIQ, J1 Conn_01x16_Socket, J14 Conn_01x02_Pin, J15 Conn_01x02_Pin, J2 USB_C_Receptacle_USB2.0_14P, J3 Conn_01x03_Socket, U13 RP2040, U14 SN74LVC244APWT, U3 74AHCT125, Y1 Crystal_12MHz

Commit message: updated RPS sch
Parts:
- renumbered C11 to C10, C12 to C11, C13 to C12, C43 to C13, C15 to C14, C14 to C15, C7 to C6, C8 to C7, C10 to C8, C6 to C9, J15 to J2, J2 to J3, J14 to J4, J3 to J5, R16 to R1, R15 to R10, R18 to R11, R60 to R12, R20 to R13, R21 to R14, R22 to R15, R23 to R16, R24 to R17, R25 to R18, R26 to R19, R17 to R2, R27 to R20, R28 to R21, R29 to R22, R30 to R23, R31 to R24, R32 to R25, R1 to R3, R2 to R4, R3 to R5, R4 to R6, R14 to R7, R5 to R8, R6 to R9, U13 to U1, U14 to U2
Connections:
- net I2C_SCL: now also U1.35 (GPIO23); no longer U1.16 (GPIO13)
- net I2C_SDA: now also U1.34 (GPIO22); no longer U1.15 (GPIO12)
- net ADC: now reaches U1.38 (GPIO26_ADC0)
- new net TPS_EN: U1.16 (GPIO13)
- no-connect marks 14 -> 13
