File: TEST V1/untitled.kicad_sch (KiCad schematic)
At the start: 14 parts, among them J5 Conn_01x01_Pin, J6 Conn_01x01_Pin, J7 Conn_01x01_Pin, J8 Conn_01x01_Pin, U9 LM2596T-5

Commit message: Integrated FG, RPS, and PCB updates
Parts:
- added C19: 10u, Capacitor_SMD:C_0603_1608Metric_Pad1.08x0.95mm_HandSolder, symbol Device:C_Small
- added C20: 100n, Capacitor_SMD:C_0603_1608Metric_Pad1.08x0.95mm_HandSolder, symbol Device:C_Small
- added C21: 0.1u, Capacitor_SMD:C_0603_1608Metric_Pad1.08x0.95mm_HandSolder, symbol Device:C_Small
- added C22, C23: 22u, Capacitor_SMD:C_0603_1608Metric_Pad1.08x0.95mm_HandSolder, symbol Device:C_Small
- added J4: Conn_01x02_Pin, Connector_PinHeader_2.54mm:PinHeader_1x01_P2.54mm_Horizontal, symbol Connector:Conn_01x02_Pin
- added J5: ~, Connector_PinHeader_2.54mm:PinHeader_1x01_P2.54mm_Vertical, symbol Connector:Conn_01x01_Pin
- added J6: Conn_01x02_Pin, symbol Connector:Conn_01x02_Pin
- added L1: 16u, Inductor_THT:L_Radial_D8.7mm_P5.00mm_Fastron_07HCP, symbol Device:L_Iron_Small
- added R33: 100k, Resistor_SMD:R_0603_1608Metric_Pad0.98x0.95mm_HandSolder, symbol Device:R_Small
- added R34: 190k, Resistor_SMD:R_0603_1608Metric_Pad0.98x0.95mm_HandSolder, symbol Device:R_Small
- added R35: 10k, Resistor_SMD:R_0603_1608Metric_Pad0.98x0.95mm_HandSolder, symbol Device:R_Small
- added U4: TPS54202DDC, Package_TO_SOT_SMD:SOT-23-6, symbol Regulator_Switching:TPS54202DDC
- added U5: MCP4725A2T-ECH, Package_TO_SOT_SMD:SOT-23-6, symbol Analog_DAC:MCP4725xxx-xCH
- R36: renamed from R24; footprint (none) -> Resistor_SMD:R_0603_1608Metric_Pad0.98x0.95mm_HandSolder
- R37: renamed from R25; footprint (none) -> Resistor_SMD:R_0603_1608Metric_Pad0.98x0.95mm_HandSolder
- R38: renamed from R27; footprint (none) -> Resistor_SMD:R_0603_1608Metric_Pad0.98x0.95mm_HandSolder
- R39: renamed from R28; footprint (none) -> Resistor_SMD:R_0603_1608Metric_Pad0.98x0.95mm_HandSolder
- R40: renamed from R29; footprint (none) -> Resistor_SMD:R_0603_1608Metric_Pad0.98x0.95mm_HandSolder
- renumbered C18 to C24, C19 to C25, D2 to D1, J8 to J10, J5 to J7, J6 to J8, J7 to J9, U9 to U6
Connections:
- net GND: now also C19.2, C20.2, C22.2, C23.2, J4.2 (Pin_2), J6.2 (Pin_2), R33.2, R35.2, U4.1 (GND), U5.2 (VSS)
- new net: C21.1, U4.6 (BOOT)
- new net: C21.2, L1.1, U4.2 (SW)
- new net: C19.1, C20.1, J4.1 (Pin_1), U4.3 (VIN)
- new net +3.3V: U5.3 (VDD), U5.6 (A0)
- new net EN: J5.1 (Pin_1), R33.1, U4.5 (EN)
- new net I2C_SCL: U5.5 (SCL)
- new net I2C_SDA: U5.4 (SDA)
- new net RPS_VOUT: C22.1, C23.1, J6.1 (Pin_1), L1.2, R34.1
- new net TPS_FB: R34.2, R35.1, U4.4 (FB), U5.1 (VOUT)
Other:
- note added: "REGULATED POWER SUPPLY"
- moved on the sheet: C24, C25, D1, J10, J7, J8, J9, L2, R36, R37, R38, R39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

Commit message: updated RPS schematic
Parts:
- removed C19: 10u, Capacitor_SMD:C_0603_1608Metric_Pad1.08x0.95mm_HandSolder, symbol Device:C_Small
- removed C20: 100n, Capacitor_SMD:C_0603_1608Metric_Pad1.08x0.95mm_HandSolder, symbol Device:C_Small
- removed C21: 0.1u, Capacitor_SMD:C_0603_1608Metric_Pad1.08x0.95mm_HandSolder, symbol Device:C_Small
- removed C22, C23: 22u, Capacitor_SMD:C_0603_1608Metric_Pad1.08x0.95mm_HandSolder, symbol Device:C_Small
- removed J4: Conn_01x02_Pin, Connector_PinHeader_2.54mm:PinHeader_1x01_P2.54mm_Horizontal, symbol Connector:Conn_01x02_Pin
- removed J5: ~, Connector_PinHeader_2.54mm:PinHeader_1x01_P2.54mm_Vertical, symbol Connector:Conn_01x01_Pin
- removed J6: Conn_01x02_Pin, symbol Connector:Conn_01x02_Pin
- removed L1: 16u, Inductor_THT:L_Radial_D8.7mm_P5.00mm_Fastron_07HCP, symbol Device:L_Iron_Small
- removed R33: 100k, Resistor_SMD:R_0603_1608Metric_Pad0.98x0.95mm_HandSolder, symbol Device:R_Small
- removed R34: 190k, Resistor_SMD:R_0603_1608Metric_Pad0.98x0.95mm_HandSolder, symbol Device:R_Small
- removed R35: 10k, Resistor_SMD:R_0603_1608Metric_Pad0.98x0.95mm_HandSolder, symbol Device:R_Small
- removed U4: TPS54202DDC, Package_TO_SOT_SMD:SOT-23-6, symbol Regulator_Switching:TPS54202DDC
- removed U5: MCP4725A2T-ECH, Package_TO_SOT_SMD:SOT-23-6, symbol Analog_DAC:MCP4725xxx-xCH
Other:
- note removed: "REGULATED POWER SUPPLY"
