File: TEST V1/untitled.kicad_sch (KiCad schematic)
At the start: 28 parts, among them J10 Conn_01x01_Pin, J4 Conn_01x02_Pin, J6 Conn_01x02_Pin, J7 Conn_01x01_Pin, J8 Conn_01x01_Pin, J9 Conn_01x01_Pin, U4 TPS54202DDC, U5 MCP4725A2T-ECH, U6 LM2596T-5

Commit message: all updated
Parts:
- J6: footprint (none) -> Connector_PinHeader_2.54mm:PinHeader_1x01_P2.54mm_Horizontal
Changed lines of the file:
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@@
 			)
 		)
-		(property "Footprint" ""
+		(property "Footprint" "Connector_PinHeader_2.54mm:PinHeader_1x01_P2.54mm_Horizontal"
 			(at 142.24 109.22 0)
 			(effects
