File: TEST V1/untitled.kicad_sch (KiCad schematic)
At the start: 14 parts, among them J10 Conn_01x01_Pin, J7 Conn_01x01_Pin, J8 Conn_01x01_Pin, J9 Conn_01x01_Pin, U6 LM2596T-5

Commit message: updated RPS sch
Parts:
- renumbered C24 to C19, C25 to C20, J7 to J6, J8 to J7, J9 to J8, J10 to J9, L2 to L1, R36 to R26, R37 to R27, R38 to R28, R39 to R29, R40 to R30, U6 to U4
Changed lines of the file:
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@@
 		(on_board yes)
 		(dnp no)
-		(property "Reference" "J8"
+		(property "Reference" "J7"
 			(at 158.115 66.04 0)
 			(effects
@@
 			(project "TEST V1"
 				(path "/e198004f-db65-4a52-ae89-6b1c9a9775ee/5cc10699-6105-455c-9975-9ca0b906834c"
-					(reference "J8")
+					(reference "J7")
 					(unit 1)
 				)
@@
 		(dnp no)
 		(fields_autoplaced yes)
-		(property "Reference" "R37"
+		(property "Reference" "R27"
 			(at 185.42 46.99 90)
 			(effects
@@
 			(project "TEST V1"
 				(path "/e198004f-db65-4a52-ae89-6b1c9a9775ee/5cc10699-6105-455c-9975-9ca0b906834c"
-					(reference "R37")
+					(reference "R27")
 					(unit 1)
 				)
@@
 		(on_board yes)
 		(dnp no)
-		(property "Reference" "J10"
+		(property "Reference" "J9"
 			(at 263.525 76.2 0)
 			(effects
@@
 			(project "TEST V1"
 				(path "/e198004f-db65-4a52-ae89-6b1c9a9775ee/5cc10699-6105-455c-9975-9ca0b906834c"
-					(reference "J10")
+					(reference "J9")
 					(unit 1)
 				)
@@
 		(on_board yes)
 		(dnp no)
-		(property "Reference" "J9"
+		(property "Reference" "J8"
 			(at 263.525 63.5 0)
 			(effects
@@
 			(project "TEST V1"
 				(path "/e198004f-db65-4a52-ae89-6b1c9a9775ee/5cc10699-6105-455c-9975-9ca0b906834c"
-					(reference "J9")
+					(reference "J8")
 					(unit 1)
 				)
@@
 		(on_board yes)
 		(dnp no)
-		(property "Reference" "R38"
+		(property "Reference" "R28"
 			(at 219.71 61.722 90)
 			(effects
@@
 			(project "TEST V1"
 				(path "/e198004f-db65-4a52-ae89-6b1c9a9775ee/5cc10699-6105-455c-9975-9ca0b906834c"
-					(reference "R38")
+					(reference "R28")
 					(unit 1)
 				)
@@
 		(dnp no)
 		(fields_autoplaced yes)
-		(property "Reference" "#PWR052"
+		(property "Reference" "#PWR049"
 			(at 205.74 82.55 0)
 			(effects
@@
 			(project "TEST V1"
 				(path "/e198004f-db65-4a52-ae89-6b1c9a9775ee/5cc10699-6105-455c-9975-9ca0b906834c"
-					(reference "#PWR052")
+					(reference "#PWR049")
 					(unit 1)
 				)
@@
 		(dnp no)
 		(fields_autoplaced yes)
-		(property "Reference" "R39"
+		(property "Reference" "R29"
 			(at 231.14 46.99 90)
 			(effects
@@
 			(project "TEST V1"
 				(path "/e198004f-db65-4a52-ae89-6b1c9a9775ee/5cc10699-6105-455c-9975-9ca0b906834c"
-					(reference "R39")
+					(reference "R29")
 					(unit 1)
 				)
@@
 		(dnp no)
 		(fields_autoplaced yes)
-		(property "Reference" "J7"
+		(property "Reference" "J6"
 			(at 158.115 48.26 0)
 			(effects
@@
 			(project "TEST V1"
 				(path "/e198004f-db65-4a52-ae89-6b1c9a9775ee/5cc10699-6105-455c-9975-9ca0b906834c"
-					(reference "J7")
+					(reference "J6")
 					(unit 1)
 				)
@@
 		(dnp no)
 		(fields_autoplaced yes)
-		(property "Reference" "U6"
+		(property "Reference" "U4"
 			(at 205.74 45.72 0)
 			(effects
@@
 			(project "TEST V1"
 				(path "/e198004f-db65-4a52-ae89-6b1c9a9775ee/5cc10699-6105-455c-9975-9ca0b906834c"
-					(reference "U6")
+					(reference "U4")
 					(unit 1)
 				)
@@
 		(on_board yes)
 		(dnp no)
-		(property "Reference" "L2"
+		(property "Reference" "L1"
 			(at 238.76 55.118 90)
 			(effects
@@
 			(project "TEST V1"
 				(path "/e198004f-db65-4a52-ae89-6b1c9a9775ee/5cc10699-6105-455c-9975-9ca0b906834c"
-					(reference "L2")
+					(reference "L1")
 					(unit 1)
 				)
@@
 		(on_board yes)
 		(dnp no)
-		(property "Reference" "#FLG04"
+		(property "Reference" "#FLG05"
 			(at 191.77 51.435 0)
 			(effects
@@
 			(project "TEST V1"
 				(path "/e198004f-db65-4a52-ae89-6b1c9a9775ee/5cc10699-6105-455c-9975-9ca0b906834c"
-					(reference "#FLG04")
+					(reference "#FLG05")
 					(unit 1)
 				)
@@
 		(on_board yes)
 		(dnp no)
-		(property "Reference" "R40"
+		(property "Reference" "R30"
 			(at 251.968 60.706 90)
 			(effects
@@
 			(project "TEST V1"
 				(path "/e198004f-db65-4a52-ae89-6b1c9a9775ee/5cc10699-6105-455c-9975-9ca0b906834c"
-					(reference "R40")
+					(reference "R30")
 					(unit 1)
 				)
@@
 		(on_board yes)
 		(dnp no)
-		(property "Reference" "C24"
+		(property "Reference" "C19"
 			(at 172.974 60.452 0)
 			(effects
@@
 			(project "TEST V1"
 				(path "/e198004f-db65-4a52-ae89-6b1c9a9775ee/5cc10699-6105-455c-9975-9ca0b906834c"
-					(reference "C24")
+					(reference "C19")
 					(unit 1)
 				)
@@
 		(on_board yes)
 		(dnp no)
-		(property "Reference" "C25"
+		(property "Reference" "C20"
 			(at 243.84 62.23 0)
 			(effects
@@
 			(project "TEST V1"
 				(path "/e198004f-db65-4a52-ae89-6b1c9a9775ee/5cc10699-6105-455c-9975-9ca0b906834c"
-					(reference "C25")
+					(reference "C20")
 					(unit 1)
 				)
@@
 		(on_board yes)
 		(dnp no)
-		(property "Reference" "R36"
+		(property "Reference" "R26"
 			(at 170.18 46.99 90)
 			(effects
@@
 			(project "TEST V1"
 				(path "/e198004f-db65-4a52-ae89-6b1c9a9775ee/5cc10699-6105-455c-9975-9ca0b906834c"
-					(reference "R36")
-					(unit 1)
-				)
+					(reference "R26")
+					(unit 1)
+				)
