File: TEST V1/RPS.kicad_sch (KiCad schematic)
At the start: 0 parts

Commit message: Integrated FG, RPS, and PCB updates
Parts:
- added C38: 10u, Capacitor_SMD:C_0603_1608Metric_Pad1.08x0.95mm_HandSolder, symbol Device:C_Small
- added C39: 100n, Capacitor_SMD:C_0603_1608Metric_Pad1.08x0.95mm_HandSolder, symbol Device:C_Small
- added C40: 0.1u, Capacitor_SMD:C_0603_1608Metric_Pad1.08x0.95mm_HandSolder, symbol Device:C_Small
- added C41, C42: 22u, Capacitor_SMD:C_0603_1608Metric_Pad1.08x0.95mm_HandSolder, symbol Device:C_Small
- added J11: Conn_01x02_Pin, Connector_PinHeader_2.54mm:PinHeader_1x01_P2.54mm_Horizontal, symbol Connector:Conn_01x02_Pin
- added J12: ~, Connector_PinHeader_2.54mm:PinHeader_1x01_P2.54mm_Vertical, symbol Connector:Conn_01x01_Pin
- added J13: Conn_01x02_Pin, symbol Connector:Conn_01x02_Pin
- added L3: 16u, Inductor_THT:L_Radial_D8.7mm_P5.00mm_Fastron_07HCP, symbol Device:L_Iron_Small
- added R57: 100k, Resistor_SMD:R_0603_1608Metric_Pad0.98x0.95mm_HandSolder, symbol Device:R_Small
- added R58: 190k, Resistor_SMD:R_0603_1608Metric_Pad0.98x0.95mm_HandSolder, symbol Device:R_Small
- added R59: 10k, Resistor_SMD:R_0603_1608Metric_Pad0.98x0.95mm_HandSolder, symbol Device:R_Small
- added U11: TPS54202DDC, Package_TO_SOT_SMD:SOT-23-6, symbol Regulator_Switching:TPS54202DDC
- added U12: MCP4725A2T-ECH, Package_TO_SOT_SMD:SOT-23-6, symbol Analog_DAC:MCP4725xxx-xCH
Connections:
- new net: C38.1, C39.1, J11.1 (Pin_1), U11.3 (VIN)
- new net: C40.2, L3.1, U11.2 (SW)
- new net: C40.1, U11.6 (BOOT)
- new net +3.3V: U12.3 (VDD), U12.6 (A0)
- new net EN: J12.1 (Pin_1), R57.1, U11.5 (EN)
- new net GND: C38.2, C39.2, C41.2, C42.2, J11.2 (Pin_2), J13.2 (Pin_2), R57.2, R59.2, U11.1 (GND), U12.2 (VSS)
- new net I2C_SCL: U12.5 (SCL)
- new net I2C_SDA: U12.4 (SDA)
- new net RPS_VOUT: C41.1, C42.1, J13.1 (Pin_1), L3.2, R58.1
- new net TPS_FB: R58.2, R59.1, U11.4 (FB), U12.1 (VOUT)
Other:
- note added: "ADDRESS= 0x61"
- note added: "REGULATED POWER SUPPLY"

Commit message: all updated
Parts:
- J13: footprint (none) -> Connector_PinHeader_2.54mm:PinHeader_1x01_P2.54mm_Horizontal
Changed lines of the file:
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@@
 			)
 		)
-		(property "Footprint" ""
+		(property "Footprint" "Connector_PinHeader_2.54mm:PinHeader_1x01_P2.54mm_Horizontal"
 			(at 185.42 60.96 0)
 			(effects
