File: TEST V1/TEST V1.kicad_pcb (KiCad board)
At the start: 2 copper layers, 125 parts, among them J1 Conn_01x16_Socket, J10 Conn_01x01_Pin, J11 Conn_01x02_Pin, J2 USB_C_Receptacle_USB2.0_14P, J3 Conn_01x03_Socket, J4 Conn_01x02_Pin, J7 Conn_01x01_Pin, J8 Conn_01x01_Pin, J9 Conn_01x01_Pin, U1 RP2040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

Commit message: all updated
Parts:
- removed U1: RP2040, Package_DFN_QFN:QFN-56-1EP_7x7mm_P0.4mm_EP3.2x3.2mm
- added C43: 100n, Capacitor_SMD:C_0603_1608Metric_Pad1.08x0.95mm_HandSolder, F.Cu at (105.1, 220.6)
- added IC1: W25Q16JVUXIQ, W25Q16JVUXIQ:SON50P300X200X60-9N, F.Cu at (137.4, 215.3)
- added J13: Conn_01x02_Pin, Connector_PinHeader_2.54mm:PinHeader_1x01_P2.54mm_Horizontal, F.Cu at (50.1, 68.3)
- added J14: Conn_01x02_Pin, Connector_PinHeader_2.54mm:PinHeader_1x02_P2.54mm_Vertical, F.Cu at (140.7, 236.9)
- added J15: Conn_01x02_Pin, Connector_PinHeader_2.54mm:PinHeader_1x02_P2.54mm_Vertical, F.Cu at (136.0, 204.5)
- added J6: Conn_01x02_Pin, Connector_PinHeader_2.54mm:PinHeader_1x01_P2.54mm_Horizontal, F.Cu at (50.1, 50.2)
- added L2: 33u, 1274AS-H-150M_P3:IND_1274AS-H-150M=P3, F.Cu at (54.7, 58.3)
- added R60: 0, Resistor_SMD:R_0603_1608Metric_Pad0.98x0.95mm_HandSolder, F.Cu at (101.4, 220.6)
- added U13: RP2040, Package_DFN_QFN:QFN-56-1EP_7x7mm_P0.4mm_EP3.2x3.2mm, F.Cu at (139.9, 222.9)
- added U14: SN74LVC244APWT, SN74LVC244APWT:SOP65P640X120-20N, F.Cu at (108.9, 227.3)
- added Y2: 25 MHz, C3E-16.000-12-1015-X-M:XTAL_C3E-16.000-12-1015-X-M, F.Cu at (66.2, 63.9)
- moved J1 161.5 mm to (54.9, 234.7), turned to 180 degrees
- moved R1 150.6 mm to (132.3, 218.5), turned to 180 degrees
- moved R28 149.0 mm to (136.7, 236.8)
- moved R14 142.0 mm to (147.3, 217.7)
- moved R3 140.5 mm to (134.9, 209.8)
- moved R2 139.7 mm to (135.1, 207.6)
- moved R4 136.9 mm to (131.8, 208.1), turned to 90 degrees
- moved R22 126.7 mm to (86.5, 216.2), turned to 180 degrees
- moved R23 122.5 mm to (86.5, 211.8), turned to 180 degrees
- moved C3 121.4 mm to (145.1, 215.8)
- moved C2 120.5 mm to (132.2, 216.7), turned to 180 degrees
- moved C1 120.2 mm to (132.3, 213.9)
- moved R24 118.2 mm to (86.8, 207.2), turned to 180 degrees
- moved R25 114.5 mm to (86.7, 203.1), turned to 180 degrees
- moved R31 107.7 mm to (117.9, 200.0), turned to 180 degrees
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Connections:
- net /ADC_AVDD renamed ADC_AVDD
- C1 pad 1: Net-(IC1-VCC) -> GND
- C1 pad 2: GND -> Net-(IC1-VCC)
- C10 pad 1: /IOVDD -> Net-(U13-USB_VDD)
- C11 pad 1: /IOVDD -> Net-(U13-USB_VDD)
- C12 pad 1: /IOVDD -> Net-(U13-USB_VDD)
- C13 pad 1: /IOVDD -> Net-(U13-USB_VDD)
- C7 pad 1: /IOVDD -> Net-(U13-USB_VDD)
- C8 pad 1: /IOVDD -> Net-(U13-USB_VDD)
- R18 pad 2: /IOVDD -> Net-(U13-USB_VDD)
- R5 pad 2: /USB_DM -> /USB_DP
- R6 pad 2: /USB_DP -> /USB_DM
- U3 pad 12: /GPIO3 -> /GPIO11
- U3 pad 2: /GPIO0 -> /GPIO8
- U3 pad 5: /GPIO1 -> /GPIO9
- U3 pad 9: /GPIO2 -> /GPIO10
Routing:
- net /QSPI_SD0: track 0.00 -> 5.80 mm
- net /QSPI_CSN: track 0.00 -> 3.32 mm
- net /QSPI_SD1: track 0.00 -> 2.98 mm
- net /QSPI_SD2: track 0.00 -> 2.94 mm
- net (no net): vias 0 -> 7
